File: pcb_quadrotor.kicad_pcb (KiCad board)
At the start: 4 copper layers, 45.2 x 60 mm, 85 parts, among them J1 Conn_01x24, J10 Conn_01x03, J11 Conn_01x03, J12 Conn_01x03, J2 Conn_01x06, J3 Conn_01x02, J4 Conn_01x03, J5 Conn_01x03, J6 Conn_01x03, J7 Conn_01x03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

Commit message: add images/docs/mechanical and Readme
Signed-off-by: ncerzzk <huangzzk@bupt.edu.cn>
Connections:
- net /SD_DATA0 renamed /D5
- net /SD_DATA1 renamed /PCLK
- C13 pad 1: Net-(C13-Pad1) -> 5V
- C14 pad 1: Net-(C13-Pad1) -> 5V
- U5 pad 5: Net-(C13-Pad1) -> 5V
Routing:
- net 5V: track 130.2 -> 146.2 mm, vias 3 -> 4
- net Net-(C13-Pad1): track 6.71 -> 0.00 mm
