File: pcb_quadrotor.kicad_sch (KiCad schematic)
At the start: 13 parts, among them J1 Conn_01x24, Q1 Q_NPN_BEC, Q2 Q_NPN_BEC, U1 E32-900M20S, U2 ESP32-WROOM-32

Commit message: add images/docs/mechanical and Readme
Signed-off-by: ncerzzk <huangzzk@bupt.edu.cn>
Other:
- note added: "IO12(MTDI should not pull up, because it determines the voltage level of VDD_SDIO, 1 for 1V8, 0 for 3V3)"
Changed lines of the file:
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@@
     (stroke (width 0) (type default) (color 0 0 0 0))
+  )
+  (text "IO12(MTDI should not pull up, \nbecause it determines the voltage level of VDD_SDIO,\n1 for 1V8, 0 for 3V3)"
+    (at 220.98 97.155 0)
+    (effects (font (size 1.27 1.27)) (justify left bottom))
   )
   (label "SCL" (at 202.565 107.315 0)
